File: Eagle_Files/PICrouter.sch (EAGLE design)
At the start: 82 parts, among them IC1 PIC32MX675F512H, IC2 48M033F, IC3 DP83848, IC4 TPS2111A, J1 POWER_JACK, Q1 20MHz, U2 DEVICE, X2 USB-A-H

Commit message: Released PICrouter schematic and board v0.93.
Parts:
- removed C31, C32: 0.1uF, rcl:C-EUC2012
- removed R28: 400, SparkFun:RESISTOR0603-RES
- added C25: 0.1uF, rcl:C-EUC2012
- added C27: 10uF, SparkFun:CAP_POL1206
- added R7: 10k, SparkFun:RESISTOR0603-RES
- C10: value 150uF -> 0.1uF; device rcl:CPOL-USC -> rcl:C-EUC2012
- C13: value 100uF -> 0.1uF; device rcl:CPOL-USC -> rcl:C-EUC2012
- C15: value 10uF -> 0.1uF; device rcl:CPOL-USC -> rcl:C-EUC2012
- C17: value 0.1uF -> 10uF
- C18: value 0.1uF -> 100uF; device rcl:C-EUC2012 -> rcl:CPOL-USC
- C19: value 10uF -> 150uF; device rcl:CPOL-USC -> SparkFun:CAP_POL3528
- C28: value 0.1uF -> 10uF; device rcl:C-EUC2012 -> SparkFun:CAP_POL1206
- C30: value 10uF -> 0.1uF
- IC2: value 48M033F -> DP83848; device linear:7805DT -> national-semiconductor:DP83848
- IC3: value DP83848 -> TPS2111A; device national-semiconductor:DP83848 -> SparkFun:TPS2111A
- IC4: value TPS2111A -> 48M033F; device SparkFun:TPS2111A -> linear:7805DT
- J1: value POWER_JACK -> (none); device SparkFun:POWER_JACKPTH_LOCK -> pulse_j0011:J0011
- J2: value (none) -> POWER_JACK; device pulse_j0011:J0011 -> SparkFun:POWER_JACKPTH_LOCK
- R10: value 10k -> 33
- R11, R12: value 49.9 -> 1.5k
- R13, R14: value 49.9 -> 33
- R15: value 4.87k -> 33
- R18: value 33 -> 4.87k
- R19: value 33 -> 2.2k
- R2: value 33 -> 400
- R21: value 1.5k -> 33
- R22: value 2.2k -> 49.9
- R23, R24: value 33 -> 49.9
- R25: value 1.5k -> 49.9
- R3: value 100 -> 330
- R4: value 10k -> 330
- R6: value 10k -> 100
- R8, R9: value 330 -> 10k
- renumbered F2 to F1
Connections:
- net ECRSDV: now also IC2.CRS; no longer IC3.CRS
- net EINT: now also IC2.PWRDN_INTN, R12.1; no longer IC3.PWRDN_INTN, R21.1
- net EMDC: now also IC2.MDC; no longer IC3.MDC
- net EMDIO: now also IC2.MDIO, R11.2; no longer IC3.MDIO, R25.2
- net EREFCLK: now also IC2.X1, R10.2; no longer IC3.X1, R2.2
- net ERXD0: now also R20.1; no longer R23.1
- net ERXD1: now also R21.1; no longer R24.1
- net ERXERR: now also IC2.RX_ER; no longer IC3.RX_ER
- net ETXD0: now also R14.1; no longer R19.1
- net ETXD1: now also R15.1; no longer R20.1
- net ETXEN: now also R13.1; no longer R18.1
- net GND: now also C10.2, C13.2, C15.2, C18.-, C25.2, C27.-, C28.-, IC2.ANA18VSS, IC2.CDVSS, IC2.CORE_VSS, IC2.IO_VSS1, IC2.IO_VSS2, IC2.TXD_3, IC3.D0, IC3.GND, IC3.VSNS, J1.CGND, J1.LC, J1.RC, J1.S1, J1.S2, J2.GND, R1.1, R18.2, R2.1; no longer C10.-, C13.-, C15.-, C18.2, C28.2, C31.2, C32.2, IC2.GND, IC3.ANA18VSS, IC3.CDVSS, IC3.CORE_VSS, IC3.IO_VSS1, IC3.IO_VSS2, IC3.TXD_3, IC4.D0, IC4.VSNS, J1.GND, J2.CGND, J2.LC, J2.RC, J2.S1, J2.S2, R15.2, R28.1, R6.1
- net LED_ACT: now also IC2.LED_ACTCOL; no longer IC3.LED_ACTCOL
- net LED_LINK: now also IC2.LED_LNK; no longer IC3.LED_LNK
- net N$10: now also R6.2; no longer R3.2
- net N$12: now also R7.2; no longer R4.2
- net N$13: now also R3.2; no longer R8.2
- net N$14: now also R4.2; no longer R9.2
- net N$15: now also R3.1; no longer R8.1
- net N$16: now also R4.1; no longer R9.1
- net N$47: now also IC2.IP_PH_P, R17.1; no longer IC3.IP_PH_P, R16.1
- net N$48: now also IC2.IP_PH_M, R16.1; no longer IC3.IP_PH_M, R17.1
- net N$49: now also IC2.RX_DV, R19.2; no longer IC3.RX_DV, R22.2
- net N$52: now also IC2.TXD_1, R15.2; no longer IC3.TXD_1, R20.2
- net N$53: now also IC2.TXD_0, R14.2; no longer IC3.TXD_0, R19.2
- net N$54: now also IC2.TX_EN, R13.2; no longer IC3.TX_EN, R18.2
- net N$55: now also J1.LA; no longer J2.LA
- net N$56: now also IC2.RXD_0, R20.2; no longer IC3.RXD_0, R23.2
- net N$57: now also IC2.RXD_1, R21.2; no longer IC3.RXD_1, R24.2
- net N$58: now also R10.1; no longer R2.1
- net N$6: now also R9.1; no longer R1.1
- net N$61: now also IC3.ILIM, R2.2; no longer IC4.ILIM, R28.2
- net N$62: now also J1.RA; no longer J2.RA
- net N$8: now also R8.1; no longer R10.1
- net N$9: now also IC2.VREF, R18.1; no longer IC3.VREF, R15.1
- net PFBOUT: now also C21.1, C22.1, C23.1, C27.+, IC2.ANA18VDD, IC2.CORE_VDD, IC2.REG_OUT; no longer C14.1, C18.1, C19.+, C20.1, IC3.ANA18VDD, IC3.CORE_VDD, IC3.REG_OUT
- net RDM: now also IC2.TPRDM, J1.RD-, R25.1; no longer IC3.TPRDM, J2.RD-, R11.1
- net RDP: now also IC2.TPRDP, J1.RD+, R24.1; no longer IC3.TPRDP, J2.RD+, R12.1
- net SELF: now also C13.1, C15.1, C16.1, IC3.D1, IC3.IN1, J2.PWR, R1.2; no longer C29.1, C31.1, C32.1, IC4.D1, IC4.IN1, J1.PWR, R6.2
- net TDM: now also IC2.TPTDM, J1.TD-, R23.1; no longer IC3.TPTDM, J2.TD-, R13.1
- net TDP: now also IC2.TPTDP, J1.TD+, R22.1; no longer IC3.TPTDP, J2.TD+, R14.1
- net VBUS: now also C14.1, C17.1, IC3.IN2, R7.1; no longer C28.1, C30.1, IC4.IN2, R4.1
- net VBUS_HOST: now also C19.+; no longer C10.+
- net VCC: now also C10.1, C18.+, IC3.OUT, IC4.VI; no longer C11.1, C13.+, IC2.VI, IC4.OUT
- net VDD: now also C11.1, C20.1, C25.1, C28.+, C29.1, C30.1, IC2.ANA33VDD, IC2.IO_VDD1, IC2.IO_VDD2, IC4.VO, J1.RCT, J1.TCT, R11.1, R19.1, R22.2, R23.2, R24.2, R25.2, R6.1, R8.2, R9.2; no longer C15.+, C16.1, C17.1, C21.1, C22.1, C23.1, IC2.VO, IC3.ANA33VDD, IC3.IO_VDD1, IC3.IO_VDD2, J2.RCT, J2.TCT, R1.2, R10.2, R11.2, R13.2, R14.2, R21.2, R22.1, R25.1, R3.1
Other:
- note added: "04/12/2012"
- note added: "PICrouter v0.93"
- note removed: "04/10/2012"
- note removed: "PICrouter v0.91"

Commit message: Released PICrouter schematic and board v0.94.
Parts:
- added S3: SSSS810701-1-2, alps_japan_potentiometers:SSSS810701-1-2
- C19: value 150uF -> 220uF; device SparkFun:CAP_POL3528 -> rcl:CPOL-USD
- C28: device SparkFun:CAP_POL1206 -> rcl:CPOL-USC
- Q1: device crystal:CRYSTALCTS406 -> my-crystal:CRYSTAL
- QG1: value SM77H -> 50MHz; device crystal:SM77H -> my-crystal:SM77H
Connections:
- new net VBUS_DEVICE: C14.1, C17.1, IC3.IN2, R7.1, S3.P$3, U2.VBUS
- net D+: now also X2.D+; no longer X2.D-
- net D-: now also X2.D-; no longer X2.D+
- net GND: now also S3.P$4, S3.P$5, S3.P$6, S3.P$7, X2.GND; no longer J1.LC, J1.RC, X2.VBUS
- net LED_ACT: now also J1.RC; no longer R27.1
- net LED_LINK: now also J1.LC; no longer R26.1
- net VBUS: now also S3.P$2; no longer C14.1, C17.1, IC3.IN2, R7.1, U2.VBUS
- net VBUS_HOST: now also S3.P$1, X2.VBUS; no longer X2.GND
- net VDD: now also R26.1, R27.1
Other:
- note added: "05/15/2012"
- note added: "PICrouter v0.95"
- note removed: "04/12/2012"
- note removed: "PICrouter v0.93"
- moved on the sheet: R26, R27

Commit message: PICrouter sch/brd v1.0 is released.
Parts:
- removed 3.3V: (no value), SparkFun:M03PTH
- removed S3: SSSS810701-1-2, alps_japan_potentiometers:SSSS810701-1-2
- added 3V3: (no value), SparkFun:M04PTH
- 5V, GND: device SparkFun:M03PTH -> SparkFun:M04PTH
- C27: device SparkFun:CAP_POL1206 -> SparkFun:CAP_POL6032
- F1: value PTCSMD -> PTC
- R2: value 400 -> 402
- renumbered AN to ANALOG, I/O to DI/O, OC to PWM
Connections:
- removed net VBUS_HOST: C19.+, F1.2, S3.P$1, X2.VBUS
- net GND: now also GND.4; no longer S3.P$4, S3.P$5, S3.P$6, S3.P$7
- net VBUS: now also C19.+, F1.2, X2.VBUS; no longer S3.P$2
- net VBUS_DEVICE: no longer S3.P$3
- net VCC: now also 5V.4
- net VDD: now also 3V3.1, 3V3.2, 3V3.3, 3V3.4; no longer 3.3V.1, 3.3V.2, 3.3V.3
Other:
- note added: "PICrouter v0.96"
- note removed: "PICrouter v0.95"
